File: electric-chair.kicad_sch (KiCad schematic)
At the start: 53 parts, among them J2 MAX632ACSA+, J3 SELFPROG, Q1 DMN2310U-7, Q2 FDN302P, Q3 IRFML8244TRPBF, Q4 NTR0202PL, Q5 DMN2310U-7, Q6 IRFML8244TRPBF, Q7 DMN2310U-7, SW1 PROGRAM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

Commit message: Docs
Parts:
- U1: value AVR32DB28x-xSO -> AVRxDB32; symbol MCU_Microchip_AVR_Dx:AVR32DB32x-xPT -> MCU_Microchip_AVR_Dx:AVR128DB32x-xPT
Changed lines of the file:
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@@
     )
   )
-  (symbol (lib_id "MCU_Microchip_AVR_Dx:AVR32DB32x-xPT") (at 80.01 66.04 0) (unit 1)
+  (symbol (lib_id "MCU_Microchip_AVR_Dx:AVR128DB32x-xPT") (at 80.01 66.04 0) (unit 1)
     (in_bom yes) (on_board yes) (dnp no)
     (property "Reference" "U1" (at 82.2041 93.98 0)
       (effects (font (size 1.27 1.27)) (justify left))
     )
-    (property "Value" "AVR32DB28x-xSO" (at 86.36 93.98 0)
+    (property "Value" "AVRxDB32" (at 86.36 93.98 0)
       (effects (font (size 1.27 1.27)) (justify left))
     )
@@
       (effects (font (size 1.27 1.27) italic) hide)
     )
-    (property "Datasheet" "https://ww1.microchip.com/downloads/en/DeviceDoc/AVR32DB28-32-48-DataSheet-DS40002301A.pdf" (at 80.01 66.04 0)
+    (property "Datasheet" "https://ww1.microchip.com/downloads/en/DeviceDoc/AVR128DB28-32-48-64-DataSheet-DS40002247A.pdf" (at 80.01 66.04 0)
       (effects (font (size 1.27 1.27)) hide)
     )

Commit message: Value fixes
Parts:
- L1: value 150uH -> 330uH
Other:
- note added: "As in prototype: D4: green 1206 led R4=560Ω Vf(D4)=2V I(R4,D4)=5.5mA"
- note added: "This circuit should provide around 10 mA of current. When not installed, 12V can be fed through TP1."
- note removed: "As in prototype: D4: red 1206 led R4=1800Ω Vf(D4)=1.8V"
- note removed: "This circuit should provide around 25 mA of usable current. When not installed, 12V can be fed through TP1, although it has to be externally fused at around 50mA."
Changed lines of the file:
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@@
     (fill (type none))
   )
-  (text "This circuit should provide around 25 mA of usable current. \nWhen not installed, 12V can be fed through TP1, although\nit has to be externally fused at around 50mA."
-    (at 15.24 113.03 0)
+  (text "This circuit should provide around 10 mA of current. \nWhen not installed, 12V can be fed through TP1."
+    (at 15.24 110.49 0)
     (effects (font (size 1.27 1.27)) (justify left bottom))
   )
@@
     (effects (font (size 1.27 1.27)) (justify left bottom))
   )
-  (text "As in prototype:\nD4: red 1206 led\nR4=1800Ω\nVf(D4)=1.8V"
+  (text "As in prototype:\nD4: green 1206 led\nR4=560Ω\nVf(D4)=2V\nI(R4,D4)=5.5mA"
     (at 26.67 170.18 0)
     (effects (font (size 1.27 1.27)) (justify left bottom))
@@
       (effects (font (size 1.27 1.27)))
     )
-    (property "Value" "150uH" (at 63.5 115.57 90)
-      (effects (font (size 1.27 1.27)))
-    )
+    (property "Value" "330uH" (at 63.5 115.57 90)
+      (effects (font (size 1.27 1.27)))
+    )
